File: Eagle/HamMessenger Shield/Shield.sch (EAGLE design)
At the start: 22 parts, among them J2 KEYBOARD GROVE, Q1 2N7000

Commit message: Continue work on PCB. Update schematic.
Parts:
- removed C2: 4.7uF, resistor:CPOL-EUE2.5-5V
- removed Q1: 2N7000, transistor-fet-edited:2N3820
- removed R1, R6: 1k, resistor:R-EU_0204/2V
- removed R2: 2k2, resistor:R-EU_0204/2V
- removed R3: 3k9, resistor:R-EU_0204/2V
- removed R4: 8k2, resistor:R-EU_0204/2V
- removed R7: 270, resistor:R-EU_0204/2V
- added C3: 100nf, Capacitor:C_CHIP-0805(2012-METRIC)
- added M1: ARDUINO-PRO-MINI-3.3V, diy-modules:ARDUINO-PRO-MINI-3.3V
- added Q3: MOSFET-NCHANNEL2N7002PW, BeagleBone_Blue_R3:MOSFET-NCHANNEL2N7002PW
- added R13: 2k2, Resistor:R_CHIP-0805(2012-METRIC)
- added R14: 3k9, Resistor:R_CHIP-0805(2012-METRIC)
- added R15: 8k2, Resistor:R_CHIP-0805(2012-METRIC)
- added R16: 1k, Resistor:R_CHIP-0805(2012-METRIC)
- added R17: 270, Resistor:R_CHIP-0805(2012-METRIC)
- added R8: 10k, Resistor:R_CHIP-0805(2012-METRIC)
- C1: value 100nF -> 4.7uf; device capacitor-wima:C2.5/2 -> adafruit:CPOL-USCT3528
- R9: value 10k -> 1k; device rcl:R-EU_0204/2V -> Resistor:R_CHIP-0805(2012-METRIC)
Connections:
- new net RX_GPS: IC1.PJ0(RXD3/PCINT9), U$1.TXD
- new net RX_MODEM: IC1.(RXD1/INT2)PD2, M1.D1/TX
- new net TX_GPS: IC1.PJ1(TXD3/PCINT10), U$1.RXD
- new net TX_MODEM: IC1.(TXD1/INT3)PD3, M1.D0/RX
- new net VCC: IC1.+VIN, M1.RAW
- net A0: now also M1.A0
- net D10: now also IC1.PF5(ADC5/TMS), M1.D10
- net D3: now also M1.D3, Q3.G, R8.2; no longer Q1.G, R9.1
- net D4: now also M1.D4, R15.2; no longer R4.1
- net D5: now also M1.D5, R14.2; no longer R3.1
- net D6: now also M1.D6, R13.2; no longer R2.1
- net D7: now also M1.D7, R9.2; no longer R1.1
- net D9: now also IC1.PF6(ADC6/TDO), M1.D9
- net GND: now also C1.-, C3.1, C3.2, M1.GND.1, Q3.S, R13.1, R14.1, R15.1, R16.1, R17.1, R17.2, R8.1, R9.1; no longer C1.1, C1.2, C2.-, Q1.D, R1.2, R2.2, R3.2, R4.2, R6.1, R7.1, R7.2, R9.2
- net LINE_LEVEL_OUT: now also C1.+; no longer C2.+
- net MIC_LEVEL_OUT: now also R16.2; no longer R6.2
- net PTT_V+: now also Q3.D; no longer Q1.S
- net SCL: now also IC1.(SDA/INT1)PD1
- net SDA: now also IC1.(SCL/INT0)PD0
Other:
- moved on the sheet: R9

Commit message: Net re-routing
Connections:
- new net N$2: C1.-, C3.1, R13.1, R14.1, R15.1, R17.2, R9.1
- net GND: no longer C1.-, C3.1, R13.1, R14.1, R15.1, R17.2, R9.1

Commit message: PCB Updates
Parts:
- added J3: (no value), Wurth_Connectors_WR-TBL Rising Cage Clamp:691210910004
Connections:
- net GND: now also J3.1
- net LINE_LEVEL_IN: now also J3.4
- net MIC_LEVEL_OUT: now also J3.3
- net PTT_V+: now also J3.2
Changed lines of the file:
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@@
 <part name="C3" library="Capacitor" library_urn="urn:adsk.eagle:library:16290819" deviceset="C" device="CHIP-0805(2012-METRIC)" package3d_urn="urn:adsk.eagle:package:16290897/2" technology="_" value="100nf"/>
 <part name="C1" library="adafruit" library_urn="urn:adsk.eagle:library:420" deviceset="CPOL-US" device="CT3528" package3d_urn="urn:adsk.eagle:package:6240405/1" value="4.7uf"/>
+<part name="J3" library="Wurth_Connectors_WR-TBL Rising Cage Clamp" library_urn="urn:adsk.eagle:library:16280519" deviceset="691210910004" device="" package3d_urn="urn:adsk.eagle:package:16248430/2"/>
 </parts>
 <sheets>
@@
 <attribute name="VALUE" x="158.496" y="36.449" size="1.778" layer="96"/>
 </instance>
+<instance part="J3" gate="G$1" x="127" y="93.98" smashed="yes">
+<attribute name="NAME" x="119.58" y="93.058" size="1.016" layer="95" align="bottom-right"/>
+<attribute name="VALUE" x="119.63" y="91.4" size="1.016" layer="96" align="bottom-right"/>
+</instance>
 </instances>
 <busses>
@@
 <wire x1="162.56" y1="68.58" x2="157.48" y2="68.58" width="0.1524" layer="91"/>
 <junction x="157.48" y="68.58"/>
+</segment>
+<segment>
+<pinref part="J3" gate="G$1" pin="3"/>
+<wire x1="127" y1="88.9" x2="127" y2="68.58" width="0.1524" layer="91"/>
+<label x="127" y="68.58" size="1.778" layer="95" rot="R90"/>
 </segment>
 </net>
@@
 <junction x="175.26" y="15.24"/>
 </segment>
+<segment>
+<pinref part="J3" gate="G$1" pin="1"/>
+<wire x1="121.92" y1="88.9" x2="121.92" y2="68.58" width="0.1524" layer="91"/>
+<label x="121.92" y="68.58" size="1.778" layer="95" rot="R90"/>
+</segment>
 </net>
 <net name="LINE_LEVEL_IN" class="0">
@@
 <pinref part="C4" gate="G$1" pin="2"/>
 <label x="93.98" y="27.94" size="1.778" layer="95"/>
+</segment>
+<segment>
+<pinref part="J3" gate="G$1" pin="4"/>
+<wire x1="129.54" y1="88.9" x2="129.54" y2="68.58" width="0.1524" layer="91"/>
+<label x="129.54" y="68.58" size="1.778" layer="95" rot="R90"/>
 </segment>
 </net>
@@
 <label x="66.04" y="86.36" size="1.778" layer="95"/>
 </segment>
-</net>
+<segment>
+<pinref part="J3" gate="G$1" pin="2"/>
+<wire x1="124.46" y1="88.9" x2="124.46" y2="68.58" width="0.1524" layer="91"/>
+<label x="124.46" y="68.58" size="1.778" layer="95" rot="R90"/>
+</segment>
+</net>

Commit message: add SD card. rerouting.
Parts:
- added U$3: MICROSD, adafruit:MICROSD
- added U2: (no value), adafruit:TXB0104PWR
Connections:
- new net MISO: IC1.(MISO/PCINT3)PB3, U$3.DATA_OUT
- new net MOSI: IC1.(MOSI/PCINT2)PB2, U2.B1
- new net N$1: U$3.DATA_IN, U2.A1
- new net N$5: U$3.SCLK, U2.A2
- new net N$6: U$3.CS, U2.A3
- new net SCK: IC1.(SCK/PCINT1)PB1, U2.B2
- new net SS: IC1.(SS/PCINT0)PB0, U2.B3
- net +3V3: now also IC1.+3V3, U$3.VDD, U2.VCCA
- net +5V: now also U2.VCCB
- net GND: now also M1.GND.2, U$3.GND, U$3.GND1, U2.GND
