File: Eagle/HamMessenger Shield/Shield.sch (EAGLE design)
At the start: 26 parts, among them J2 KEYBOARD GROVE, M1 ARDUINO-PRO-MINI-3.3V, Q3 MOSFET-NCHANNEL2N7002PW

Commit message: Change pins grove keyboard connector.
Parts:
- removed IC1: (no value), arduino:MEGAARDUINO_1
- added M2: ARDUINO-PRO-MINI-3.3V, diy-modules:ARDUINO-PRO-MINI-3.3V
- M1: value ARDUINO-PRO-MINI-3.3V -> (none); device diy-modules:ARDUINO-PRO-MINI-3.3V -> arduino:MEGAARDUINO_1
- renumbered U$1 to GPS, U$2 to OLED
Connections:
- net +3V3: now also M1.+3V3; no longer IC1.+3V3
- net +5V: now also J2.3, M1.+5V@1; no longer IC1.+5V@1, J2.2
- net A0: now also M2.A0; no longer M1.A0
- net D10: now also M1.PF5(ADC5/TMS), M2.D10; no longer IC1.PF5(ADC5/TMS), M1.D10
- net D3: now also M2.D3; no longer M1.D3
- net D4: now also M2.D4; no longer M1.D4
- net D5: now also M2.D5; no longer M1.D5
- net D6: now also M2.D6; no longer M1.D6
- net D7: now also M2.D7; no longer M1.D7
- net D9: now also M1.PF6(ADC6/TDO), M2.D9; no longer IC1.PF6(ADC6/TDO), M1.D9
- net GND: now also J2.4, M1.GND@1, M2.GND.1, M2.GND.2; no longer IC1.GND@1, J2.1, M1.GND.1, M1.GND.2
- net MISO: now also M1.(MISO/PCINT3)PB3; no longer IC1.(MISO/PCINT3)PB3
- net MOSI: now also M1.(MOSI/PCINT2)PB2; no longer IC1.(MOSI/PCINT2)PB2
- net RX_GPS: now also M1.PJ0(RXD3/PCINT9); no longer IC1.PJ0(RXD3/PCINT9)
- net RX_MODEM: now also M1.(RXD1/INT2)PD2, M2.D1/TX; no longer IC1.(RXD1/INT2)PD2, M1.D1/TX
- net SCK: now also M1.(SCK/PCINT1)PB1; no longer IC1.(SCK/PCINT1)PB1
- net SCL: now also J2.1, M1.(SDA/INT1)PD1; no longer IC1.(SDA/INT1)PD1, J2.4
- net SDA: now also J2.2, M1.(SCL/INT0)PD0; no longer IC1.(SCL/INT0)PD0, J2.3
- net SS: now also M1.(SS/PCINT0)PB0; no longer IC1.(SS/PCINT0)PB0
- net TX_GPS: now also M1.PJ1(TXD3/PCINT10); no longer IC1.PJ1(TXD3/PCINT10)
- net TX_MODEM: now also M1.(TXD1/INT3)PD3, M2.D0/RX; no longer IC1.(TXD1/INT3)PD3, M1.D0/RX
- net VCC: now also M1.+VIN, M2.RAW; no longer IC1.+VIN, M1.RAW
Other:
- moved on the sheet: J2

Commit message: Last minute tweeks before sending to fab.
Parts:
- renumbered U$3 to SD
Changed lines of the file:
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@@
 <part name="C1" library="adafruit" library_urn="urn:adsk.eagle:library:420" deviceset="CPOL-US" device="CT3528" package3d_urn="urn:adsk.eagle:package:6240405/1" value="4.7uf"/>
 <part name="J3" library="Wurth_Connectors_WR-TBL Rising Cage Clamp" library_urn="urn:adsk.eagle:library:16280519" deviceset="691210910004" device="" package3d_urn="urn:adsk.eagle:package:16248430/2"/>
-<part name="U$3" library="adafruit" library_urn="urn:adsk.eagle:library:420" deviceset="MICROSD" device="" package3d_urn="urn:adsk.eagle:package:6240723/1"/>
+<part name="SD" library="adafruit" library_urn="urn:adsk.eagle:library:420" deviceset="MICROSD" device="" package3d_urn="urn:adsk.eagle:package:6240723/1"/>
 <part name="U2" library="adafruit" library_urn="urn:adsk.eagle:library:420" deviceset="TXB0104PWR" device="" package3d_urn="urn:adsk.eagle:package:6240844/1"/>
 <part name="+3V2" library="supply1" library_urn="urn:adsk.eagle:library:371" deviceset="+3V3" device=""/>
@@
 <attribute name="VALUE" x="119.63" y="91.4" size="1.016" layer="96" align="bottom-right"/>
 </instance>
-<instance part="U$3" gate="G$1" x="401.32" y="137.16" smashed="yes"/>
+<instance part="SD" gate="G$1" x="401.32" y="137.16" smashed="yes"/>
 <instance part="U2" gate="G$1" x="337.82" y="139.7" smashed="yes" rot="MR0">
 <attribute name="NAME" x="350.52" y="157.48" size="1.27" layer="95" rot="MR0"/>
@@
 </segment>
 <segment>
-<pinref part="U$3" gate="G$1" pin="GND1"/>
+<pinref part="SD" gate="G$1" pin="GND1"/>
 <wire x1="383.54" y1="119.38" x2="378.46" y2="119.38" width="0.1524" layer="91"/>
-<pinref part="U$3" gate="G$1" pin="GND"/>
+<pinref part="SD" gate="G$1" pin="GND"/>
 <wire x1="383.54" y1="116.84" x2="378.46" y2="116.84" width="0.1524" layer="91"/>
 <pinref part="GND10" gate="1" pin="GND"/>
@@
 </segment>
 <segment>
-<pinref part="U$3" gate="G$1" pin="VDD"/>
+<pinref part="SD" gate="G$1" pin="VDD"/>
 <pinref part="+3V4" gate="G$1" pin="+3V3"/>
 <wire x1="383.54" y1="127" x2="370.84" y2="127" width="0.1524" layer="91"/>
@@
 <segment>
 <pinref part="U2" gate="G$1" pin="A1"/>
-<pinref part="U$3" gate="G$1" pin="DATA_IN"/>
+<pinref part="SD" gate="G$1" pin="DATA_IN"/>
 <wire x1="353.06" y1="142.24" x2="383.54" y2="142.24" width="0.1524" layer="91"/>
 </segment>
@@
 <segment>
 <pinref part="U2" gate="G$1" pin="A2"/>
-<pinref part="U$3" gate="G$1" pin="SCLK"/>
+<pinref part="SD" gate="G$1" pin="SCLK"/>
 <wire x1="353.06" y1="139.7" x2="383.54" y2="139.7" width="0.1524" layer="91"/>
 </segment>
@@
 <segment>
 <pinref part="U2" gate="G$1" pin="A3"/>
-<pinref part="U$3" gate="G$1" pin="CS"/>
+<pinref part="SD" gate="G$1" pin="CS"/>
 <wire x1="353.06" y1="137.16" x2="383.54" y2="137.16" width="0.1524" layer="91"/>
 </segment>
@@
 </segment>
 <segment>
-<pinref part="U$3" gate="G$1" pin="DATA_OUT"/>
+<pinref part="SD" gate="G$1" pin="DATA_OUT"/>
 <wire x1="383.54" y1="144.78" x2="370.84" y2="144.78" width="0.1524" layer="91"/>
 <label x="370.84" y="144.78" size="1.778" layer="95"/>
