File: Eagle/HamMessenger Shield/Shield.brd (EAGLE design)
At the start: 101.9 x 53.6 mm, 26 parts, among them J2 KEYBOARD GROVE, M1 ARDUINO-PRO-MINI-3.3V, Q3 MOSFET-NCHANNEL2N7002PW

Commit message: Change pins grove keyboard connector.
Parts:
- removed IC1: (no value), arduino:MEGA_ARDUINO
- added M2: ARDUINO-PRO-MINI-3.3V, diy-modules:ARDUINO-PRO-MINI
- M1: value ARDUINO-PRO-MINI-3.3V -> (none); device diy-modules:ARDUINO-PRO-MINI -> arduino:MEGA_ARDUINO
- moved M1 82.7 mm to (0.00, 0.00), turned to 0 degrees
- renumbered U$1 to GPS, U$2 to OLED
Connections:
- net +3V3: now also M1.2; no longer IC1.2
- net +5V: now also J2.3, M1.3, M1.47, M1.48; no longer IC1.3, IC1.47, IC1.48, J2.2
- net A0: now also M2.J6.8; no longer M1.J6.8
- net D10: now also M1.12, M2.J6.12; no longer IC1.12, M1.J6.12
- net D3: now also M2.J7.7; no longer M1.J7.7
- net D4: now also M2.J7.6; no longer M1.J7.6
- net D5: now also M2.J7.5; no longer M1.J7.5
- net D6: now also M2.J7.4; no longer M1.J7.4
- net D7: now also M2.J7.3; no longer M1.J7.3
- net D9: now also M1.13, M2.J7.1; no longer IC1.13, M1.J7.1
- net GND: now also J2.4, M1.4, M1.45, M1.5, M1.81, M1.82, M2.J6.2, M2.J7.9; no longer IC1.4, IC1.45, IC1.5, IC1.81, IC1.82, J2.1, M1.J6.2, M1.J7.9
- net MISO: now also M1.77; no longer IC1.77
- net MOSI: now also M1.78; no longer IC1.78
- net RX_GPS: now also M1.29; no longer IC1.29
- net RX_MODEM: now also M1.25, M2.J7.12; no longer IC1.25, M1.J7.12
- net SCK: now also M1.79; no longer IC1.79
- net SCL: now also J2.1, M1.24; no longer IC1.24, J2.4
- net SDA: now also J2.2, M1.23; no longer IC1.23, J2.3
- net SS: now also M1.80; no longer IC1.80
- net TX_GPS: now also M1.30; no longer IC1.30
- net TX_MODEM: now also M1.26, M2.J7.11; no longer IC1.26, M1.J7.11
- net VCC: now also M1.6, M2.J6.1, M2.J6.4; no longer IC1.6, M1.J6.1, M1.J6.4
Routing:
- net GND: track 164.7 -> 58.3 mm
- net +5V: track 162.7 -> 154.0 mm, vias 0 -> 1
- net LINE_LEVEL_OUT: track 93.1 -> 90.4 mm
- net SCL: track 85.2 -> 82.8 mm
- net SDA: track 89.7 -> 88.4 mm, vias 1 -> 2
Other:
- board text added: "HamMessenger v1.0 https://github.com/dalethomas81/HamMessenger Thanks for all your support, mkt :)"
- board text removed: "HamMessenger v1.0 Special Thanks: mkt"

Commit message: Last minute tweeks before sending to fab.
Parts:
- renumbered U$3 to SD
Routing:
- net GND: track 58.3 -> 49.3 mm
- net PTT_V+: track 99.1 -> 100.1 mm
