File: Documentation/CAD/Eagle/Shield/Shield.brd (EAGLE design)
At the start: 101.9 x 53.6 mm, 26 parts, among them J2 KEYBOARD GROVE, M2 ARDUINO-PRO-MINI-3.3V, Q3 MOSFET-NCHANNEL2N7002PW

Commit message: Board fixes / improvements
Parts:
- moved J2 29.5 mm to (38.4, 43.4), flipped to the bottom, turned to 270 degrees
- moved J3 20.1 mm to (24.3, 6.39), turned to 0 degrees
- moved OLED 7.84 mm to (21.4, 31.8)
- moved SD 5.00 mm to (15.5, 16.1)
Connections:
- net +3V3: now also U2.8
- net GND: now also SD.6
- net RX_GPS: now also M1.27; no longer M1.29
- net SCL: now also M1.23; no longer M1.24
- net SDA: now also M1.24; no longer M1.23
- net TX_GPS: now also M1.28; no longer M1.30
Routing:
- net MIC_LEVEL_OUT: track 114.5 -> 87.4 mm
- net SDA: track 88.4 -> 63.0 mm, vias 2 -> 1
- net LINE_LEVEL_IN: track 121.8 -> 98.4 mm
- net SCL: track 82.8 -> 66.3 mm
- net PTT_V+: track 100.1 -> 85.0 mm, vias 4 -> 3
- net N$5: track 20.5 -> 28.0 mm
- net +5V: track 154.0 -> 161.4 mm, vias 1 -> 0
- net RX_GPS: track 48.9 -> 54.0 mm
- net +3V3: track 122.7 -> 126.0 mm, vias 3 -> 5
- net D3: track 15.3 -> 18.1 mm
- net MISO: track 109.4 -> 106.9 mm
- net SS: track 79.3 -> 81.8 mm
- net TX_GPS: track 45.8 -> 47.9 mm
- net N$1: track 15.8 -> 17.4 mm
- net N$6: track 15.5 -> 16.7 mm
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Other:
- board text added: "HamMessenger v1.1 https://github.com/dalethomas81/HamMessenger Thanks for all your support, mkt :)"
- board text removed: "HamMessenger v1.0 https://github.com/dalethomas81/HamMessenger Thanks for all your support, mkt :)"

Commit message: final touch before fab
Routing:
- net GND: track 49.3 -> 44.7 mm
Changed lines of the file:
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@@
 <drawing>
 <settings>
-<setting alwaysvectorfont="yes"/>
+<setting alwaysvectorfont="no"/>
 <setting verticaltext="up"/>
 </settings>
@@
 <wire x1="81.28" y1="19.6723" x2="81.9277" y2="19.6723" width="0.1524" layer="1"/>
 <wire x1="83.66125" y1="17.93875" x2="81.9277" y2="19.6723" width="0.1524" layer="1"/>
-<wire x1="76.2602" y1="27.07338125" x2="76.2602" y2="28.80661875" width="0.1524" layer="1"/>
-<wire x1="75.8495" y1="26.66268125" x2="76.2602" y2="27.07338125" width="0.1524" layer="1"/>
-<wire x1="75.8495" y1="24.384" x2="75.8495" y2="26.66268125" width="0.1524" layer="1"/>
 <wire x1="75.8495" y1="24.384" x2="75.946" y2="24.4805" width="0.1524" layer="1"/>
 <wire x1="77.47" y1="24.4805" x2="78.74" y2="25.7505" width="0.1524" layer="1"/>
